File: SID/C64-SwinSID/C64-SwinSID.kicad_sch (KiCad schematic)
At the start: 13 parts, among them U1 ATmega88PA-A, U2 C64_SID_6581_socket, X1 SG-7050CAN

Commit message: Addition of Cartridge/C64-Cartridge to support DIP32 EEPROMs. Addition of Interactive Boms.
Parts:
- X1: value SG-7050CAN -> 32MHz
Changed lines of the file:
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@@
       (effects (font (size 1.27 1.27)))
     )
-    (property "Value" "SG-7050CAN" (at 238.76 131.5593 0)
+    (property "Value" "32MHz" (at 238.76 131.5593 0)
       (effects (font (size 1.27 1.27)))
     )
