File: Drive/C64-Pi1541/C64-Pi1541.kicad_pcb (KiCad board)
At the start: 2 copper layers, 64.1 x 34.9 mm, 38 parts, among them J1 IEC_DIN, J2 Raspberry_Pi_2_3, J3 IEC_OUT, J4 LCD_OLED, Q1 BSS138, Q2 BSS138, Q3 BSS138, Q4 BSS138, SW1 RESET, SW2 RESET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

Commit message: Addition of Cartridge/C64-Cartridge to support DIP32 EEPROMs. Addition of Interactive Boms.
Parts:
- added J5: USB_B_Micro power, Connector_USB:USB_Micro-B_Molex-105017-0001, B.Cu at (202.2, 76.5)
- moved G*** 1.91 mm to (207.7, 76.5)
Routing:
- net GND: track 23.5 -> 31.3 mm
- net +5V: track 94.6 -> 96.8 mm
Changed lines of the file:
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@@
   (net 42 "unconnected-(U1-Pad10)")
   (net 43 "unconnected-(U1-Pad12)")
+  (net 44 "unconnected-(J5-D--Pad2)")
+  (net 45 "unconnected-(J5-D+-Pad3)")
+  (net 46 "unconnected-(J5-ID-Pad4)")
   (footprint "MountingHole:MountingHole_2.5mm" (layer "F.Cu")
     (at 260.877 86.132)
@@
     )
   )
+  (footprint "Connector_USB:USB_Micro-B_Molex-105017-0001" (layer "B.Cu")
+    (at 202.2225 76.4995 90)
+    (descr "http://www.molex.com/pdm_docs/sd/1050170001_sd.pdf")
+    (tags "Micro-USB SMD Typ-B")
+    (property "Sheetfile" "C64-Pi1541.kicad_sch")
+    (property "Sheetname" "")
+    (property "ki_description" "USB Micro Type B connector")
+    (property "ki_keywords" "connector USB micro")
+    (attr smd)
+    (fp_text reference "J5" (at 0 3.1125 90) (layer "B.SilkS") hide
+        (effects (font (size 1 1) (thickness 0.15)) (justify mirror))
+    )
+    (fp_text value "USB_B_Micro power" (at 0.3 -4.3375 90) (layer "B.Fab")
+        (effects (font (size 1 1) (thickness 0.15)) (justify mirror))
+    )
+    (fp_text user "PCB Edge" (at 0 -2.6875 90) (layer "Dwgs.User")
+        (effects (font (size 0.5 0.5) (thickness 0.08)))
+    )
+    (fp_text user "${REFERENCE}" (at 0 -0.8875 90) (layer "B.Fab")
+        (effects (font (size 1 1) (thickness 0.15)) (justify mirror))
+    )
+    (fp_line (start -3.9 -2.6375) (end -3.9 -2.3875)
+      (stroke (width 0.12) (type solid)) (layer "B.SilkS"))
+    (fp_line (start -3.9 -0.0875) (end -3.9 1.7625)
+      (stroke (width 0.12) (type solid)) (layer "B.SilkS"))
+    (fp_line (start -3.9 1.7625) (end -3.45 1.7625)
+      (stroke (width 0.12) (type solid)) (layer "B.SilkS"))
+    (fp_line (start -1.7 2.3125) (end -1.7 1.8625)
+      (stroke (width 0.12) (type solid)) (layer "B.SilkS"))
+    (fp_line (start -1.7 2.3125) (end -1.25 2.3125)
+      (stroke (width 0.12) (type solid)) (layer "B.SilkS"))
+    (fp_line (start 3.9 -2.6375) (end 3.9 -2.3875)
+      (stroke (width 0.12) (type solid)) (layer "B.SilkS"))
+    (fp_line (start 3.9 -0.0875) (end 3.9 1.7625)
+      (stroke (width 0.12) (type solid)) (layer "B.SilkS"))
+    (fp_line (start 3.9 1.7625) (end 3.45 1.7625)
+      (stroke (width 0.12) (type solid)) (layer "B.SilkS"))
+    (fp_line (start -4.4 -3.64) (end -4.4 2.46)
+      (stroke (width 0.05) (type solid)) (layer "B.CrtYd"))
+    (fp_line (start -4.4 -3.64) (end 4.4 -3.64)
+      (stroke (width 0.05) (type solid)) (layer "B.CrtYd"))
+    (fp_line (start -4.4 2.46) (end 4.4 2.46)
+      (stroke (width 0.05) (type solid)) (layer "B.CrtYd"))
+    (fp_line (start 4.4 2.46) (end 4.4 -3.64)
+      (stroke (width 0.05) (type solid)) (layer "B.CrtYd"))
+    (fp_line (start -3.75 -3.389204) (end 3.75 -3.389204)
+      (stroke (width 0.1) (type solid)) (layer "B.Fab"))
+    (fp_line (start -3.75 -3.3875) (end -3.75 1.6125)
+      (stroke (width 0.1) (type solid)) (layer "B.Fab"))
+    (fp_line (start -3.75 1.6125) (end 3.75 1.6125)
+      (stroke (width 0.1) (type solid)) (layer "B.Fab"))
+    (fp_line (start -3 -2.689204) (end 3 -2.689204)
+      (stroke (width 0.1) (type solid)) (layer "B.Fab"))
+    (fp_line (start -1.5 2.1225) (end -1.5 1.9125)
+      (stroke (width 0.1) (type solid)) (layer "B.Fab"))
+    (fp_line (start -1.5 2.1225) (end -1.1 2.1225)
+      (stroke (width 0.1) (type solid)) (layer "B.Fab"))
+    (fp_line (start -1.3 1.7125) (end -1.5 1.9125)
+      (stroke (width 0.1) (type solid)) (layer "B.Fab"))
+    (fp_line (start -1.1 1.9125) (end -1.3 1.7125)
+      (stroke (width 0.1) (type solid)) (layer "B.Fab"))
+    (fp_line (start -1.1 2.1225) (end -1.1 1.9125)
+      (stroke (width 0.1) (type solid)) (layer "B.Fab"))
+    (fp_line (start 3.75 -3.3875) (end 3.75 1.6125)
+      (stroke (width 0.1) (type solid)) (layer "B.Fab"))
+    (pad "1" smd rect (at -1.3 1.4625 90) (size 0.4 1.35) (layers "B.Cu" "B.Paste" "B.Mask")
+      (net 1 "+5V") (pinfunction "VBUS") (pintype "power_out"))
+    (pad "2" smd rect (at -0.65 1.4625 90) (size 0.4 1.35) (layers "B.Cu" "B.Paste" "B.Mask")
+      (net 44 "unconnected-(J5-D--Pad2)") (pinfunction "D-") (pintype "bidirectional+no_connect"))
+    (pad "3" smd rect (at 0 1.4625 90) (size 0.4 1.35) (layers "B.Cu" "B.Paste" "B.Mask")
+      (net 45 "unconnected-(J5-D+-Pad3)") (pinfunction "D+") (pintype "bidirectional+no_connect"))
+    (pad "4" smd rect (at 0.65 1.4625 90) (size 0.4 1.35) (layers "B.Cu" "B.Paste" "B.Mask")
+      (net 46 "unconnected-(J5-ID-Pad4)") (pinfunction "ID") (pintype "passive+no_connect"))
+    (pad "5" smd rect (at 1.3 1.4625 90) (size 0.4 1.35) (layers "B.Cu" "B.Paste" "B.Mask")
+      (net 2 "GND") (pinfunction "GND") (pintype "power_out"))
+    (pad "6" thru_hole oval (at -3.5 -1.2375 270) (size 1.2 1.9) (drill oval 0.6 1.3) (layers "*.Cu" "*.Mask")
+      (net 2 "GND") (pinfunction "Shield") (pintype "passive"))
+    (pad "6" smd rect (at -2.9 -1.2375 90) (size 1.2 1.9) (layers "B.Cu" "B.Mask")
+      (net 2 "GND") (pinfunction "Shield") (pintype "passive"))
+    (pad "6" thru_hole circle (at -2.5 1.4625 90) (size 1.45 1.45) (drill 0.85) (layers "*.Cu" "*.Mask")
+      (net 2 "GND") (pinfunction "Shield") (pintype "passive"))
+    (pad "6" smd rect (at -1 -1.2375 90) (size 1.5 1.9) (layers "B.Cu" "B.Paste" "B.Mask")
+      (net 2 "GND") (pinfunction "Shield") (pintype "passive"))
+    (pad "6" smd rect (at 1 -1.2375 90) (size 1.5 1.9) (layers "B.Cu" "B.Paste" "B.Mask")
+      (net 2 "GND") (pinfunction "Shield") (pintype "passive"))
+    (pad "6" thru_hole circle (at 2.5 1.4625 90) (size 1.45 1.45) (drill 0.85) (layers "*.Cu" "*.Mask")
+      (net 2 "GND") (pinfunction "Shield") (pintype "passive"))
+    (pad "6" smd rect (at 2.9 -1.2375 90) (size 1.2 1.9) (layers "B.Cu" "B.Mask")
+      (net 2 "GND") (pinfunction "Shield") (pintype "passive"))
+    (pad "6" thru_hole oval (at 3.5 -1.2375 90) (size 1.2 1.9) (drill oval 0.6 1.3) (layers "*.Cu" "*.Mask")
+      (net 2 "GND") (pinfunction "Shield") (pintype "passive"))
+    (model "${KICAD6_3DMODEL_DIR}/Connector_USB.3dshapes/USB_Micro-B_Molex-105017-0001.wrl"
+      (offset (xyz 0 0 0))
+      (scale (xyz 1 1 1))
+      (rotate (xyz 0 0 0))
+    )
+  )
   (footprint "Resistor_SMD:R_0805_2012Metric" (layer "B.Cu")
     (at 254.737 77.737 180)
@@
   )
   (footprint "Sassa:CC_BY_NC_SA_long_silkscreen" (layer "B.Cu")
-    (at 205.842 76.467 90)
+    (at 207.747 76.467 90)
     (attr through_hole)
     (fp_text reference "G***" (at 0 0 90) (layer "B.SilkS") hide
@@
   (via (at 250.292 81.547) (size 1) (drill 0.7) (layers "F.Cu" "B.Cu") (net 1))
   (via (at 205.842 85.992) (size 1) (drill 0.7) (layers "F.Cu" "B.Cu") (net 1))
+  (segment (start 205.7795 77.7995) (end 205.842 77.737) (width 0.5) (layer "B.Cu") (net 1))
   (segment (start 254.55825 81.547) (end 255.6495 80.45575) (width 0.25) (layer "B.Cu") (net 1))
   (segment (start 250.292 81.547) (end 250.232 81.487) (width 0.5) (layer "B.Cu") (net 1))
   (segment (start 250.292 81.547) (end 251.562 82.817) (width 0.5) (layer "B.Cu") (net 1))
   (segment (start 250.292 81.547) (end 254.55825 81.547) (width 0.25) (layer "B.Cu") (net 1))
+  (segment (start 205.842 85.992) (end 205.842 77.737) (width 0.5) (layer "B.Cu") (net 1))
+  (segment (start 205.842 77.737) (end 205.842 63.767) (width 0.5) (layer "B.Cu") (net 1))
   (segment (start 251.562 82.817) (end 252.517 82.817) (width 0.5) (layer "B.Cu") (net 1))
+  (segment (start 203.685 77.7995) (end 205.7795 77.7995) (width 0.4) (layer "B.Cu") (net 1))
   (segment (start 255.6495 70.117) (end 255.6495 80.277) (width 0.25) (layer "B.Cu") (net 1))
   (segment (start 205.842 63.767) (end 207.747 61.862) (width 0.5) (layer "B.Cu") (net 1))
   (segment (start 255.6495 80.45575) (end 255.6495 80.277) (width 0.25) (layer "B.Cu") (net 1))
   (segment (start 250.232 81.487) (end 250.232 79.642) (width 0.5) (layer "B.Cu") (net 1))
-  (segment (start 205.842 85.992) (end 205.842 63.767) (width 0.5) (layer "B.Cu") (net 1))
   (segment (start 243.307 61.862) (end 244.577 63.132) (width 0.25) (layer "F.Cu") (net 2))
   (segment (start 222.987 61.862) (end 221.717 63.132) (width 0.25) (layer "F.Cu") (net 2))
@@
   (segment (start 212.827 61.862) (end 211.557 63.132) (width 0.25) (layer "F.Cu") (net 2))
   (via (at 243.942 68.847) (size 0.8) (drill 0.5) (layers "F.Cu" "B.Cu") (free) (net 2))
+  (segment (start 203.075821 78.9995) (end 201.543321 77.467) (width 0.5) (layer "B.Cu") (net 2))
+  (segment (start 201.543321 77.467) (end 200.985 77.467) (width 0.5) (layer "B.Cu") (net 2))
+  (segment (start 203.685 78.9995) (end 203.075821 78.9995) (width 0.5) (layer "B.Cu") (net 2))
+  (segment (start 201.7295 75.4995) (end 200.985 75.4995) (width 0.5) (layer "B.Cu") (net 2))
+  (segment (start 203.2295 73.9995) (end 201.7295 75.4995) (width 0.5) (layer "B.Cu") (net 2))
+  (segment (start 203.685 73.9995) (end 203.2295 73.9995) (width 0.5) (layer "B.Cu") (net 2))
+  (segment (start 203.685 75.1995) (end 203.685 73.9995) (width 0.4) (layer "B.Cu") (net 2))
   (segment (start 227.432 77.737) (end 219.177 77.737) (width 0.25) (layer "F.Cu") (net 3))
   (segment (start 227.432 77.737) (end 252.832 77.737) (width 0.25) (layer "F.Cu") (net 3))

Commit message: C64-Cartridge : addition of EpyxFastload daughter board ; some silkscreen changes. C64-KungFuFlash, C64-Pi1541 : small updates before production. New C64-efuse board that fit inside the DIN plug.
Parts:
- U1: footprint Package_SO:SO-14_5.3x10.2mm_P1.27mm -> Package_DIP:DIP-14_W7.62mm; moved to F.Cu
- moved R3 12.7 mm to (242.0, 72.7)
- moved R4 12.7 mm to (242.0, 75.2)
- moved R5 12.7 mm to (242.0, 80.3)
- moved R6 12.7 mm to (242.0, 70.1)
- moved R7 12.7 mm to (242.0, 77.7)
- moved U1 11.9 mm to (255.4, 84.1), turned to 180 degrees
- moved D1 9.53 mm to (238.2, 85.4)
- moved D2 9.53 mm to (243.9, 85.4), turned to 180 degrees
- moved R1 9.53 mm to (238.2, 85.4)
- moved R2 9.53 mm to (243.9, 85.4), turned to 180 degrees
- moved C1 2.29 mm to (251.6, 84.1)
- moved Q1 1.91 mm to (237.6, 79.6)
- moved Q2 1.27 mm to (233.8, 79.6)
- moved Q3 0.63 mm to (230.0, 79.6)
Connections:
- U1 pad 1: SRQ_OUT -> GND
- U1 pad 10: unconnected-(U1-Pad10) -> CLK
- U1 pad 11: GND -> CLK_OUT
- U1 pad 12: unconnected-(U1-Pad12) -> SRQ
- U1 pad 13: GND -> SRQ_OUT
- U1 pad 2: SRQ -> unconnected-(U1-Pad2)
- U1 pad 3: CLK_OUT -> GND
- U1 pad 4: CLK -> unconnected-(U1-Pad4)
- U1 pad 5: DATA_OUT -> GND
- U1 pad 6: DATA -> unconnected-(U1-Pad6)
- U1 pad 8: unconnected-(U1-Pad8) -> DATA
- U1 pad 9: GND -> DATA_OUT
Routing:
- net ATN: track 45.8 -> 33.1 mm
- net +5V: track 96.8 -> 88.7 mm
- net CLK: track 48.7 -> 40.9 mm, vias 3 -> 2
- net SRQ: track 47.8 -> 40.6 mm, vias 2 -> 1
- net +3.3V: track 86.0 -> 78.8 mm, vias 7 -> 6
- net DATA_OUT: track 36.0 -> 41.6 mm
- net CLK_OUT: track 35.0 -> 40.1 mm, vias 2 -> 1
- net DATA: track 53.1 -> 48.4 mm
- net RESET_IN: track 37.6 -> 40.7 mm
- net SW5: track 33.0 -> 35.9 mm
- net CLK_IN: track 43.5 -> 46.5 mm
- net SND: track 13.9 -> 16.4 mm
- net ACT: track 28.3 -> 26.0 mm
- net SRQ_OUT: track 20.3 -> 18.5 mm, vias 2 -> 0
- net DATA_IN: track 26.4 -> 25.3 mm
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Other:
- board text added: "add -"
- board text added: "down next"
- board text added: "exit -"
- board text added: "sel|start exit"
- board text added: "up prev"
