File: Drive/C64-Pi1541/C64-Pi1541.kicad_sch (KiCad schematic)
At the start: 37 parts, among them J1 IEC_DIN, J2 Raspberry_Pi_2_3, J3 IEC_OUT, J4 LCD_OLED, Q1 BSS138, Q2 BSS138, Q3 BSS138, Q4 BSS138, SW1 RESET, SW2 RESET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

Commit message: Addition of Cartridge/C64-Cartridge to support DIP32 EEPROMs. Addition of Interactive Boms.
Parts:
- added J5: USB_B_Micro power, Connector_USB:USB_Micro-B_Molex-105017-0001, symbol Connector:USB_B_Micro
Connections:
- net +5V: now also J5.1 (VBUS)
- net GND: now also J5.5 (GND), J5.6 (Shield)
- no-connect marks 13 -> 16
Changed lines of the file:
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@@
   (junction (at 156.21 120.65) (diameter 0) (color 0 0 0 0)
+  )
+  (junction (at 303.53 54.61) (diameter 0) (color 0 0 0 0)
   )
   (junction (at 55.88 26.67) (diameter 0) (color 0 0 0 0)
@@
   (no_connect (at 81.28 57.15))
   (no_connect (at 81.28 72.39))
+  (no_connect (at 311.15 46.99))
   (no_connect (at 81.28 69.85))
   (no_connect (at 81.28 64.77))
   (no_connect (at 90.17 181.61))
+  (no_connect (at 311.15 44.45))
   (no_connect (at 90.17 151.13))
   (no_connect (at 40.64 39.37))
@@
   (no_connect (at 90.17 120.65))
   (no_connect (at 40.64 36.83))
+  (no_connect (at 311.15 49.53))
   (no_connect (at 81.28 67.31))
   (no_connect (at 81.28 77.47))
@@
     (stroke (width 0) (type default))
   )
+  (wire (pts (xy 314.96 39.37) (xy 314.96 36.83))
+    (stroke (width 0) (type default))
+  )
   (wire (pts (xy 128.27 31.75) (xy 128.27 77.47))
     (stroke (width 0) (type default))
@@
   )
   (wire (pts (xy 152.4 21.59) (xy 152.4 24.13))
+    (stroke (width 0) (type default))
+  )
+  (wire (pts (xy 311.15 39.37) (xy 314.96 39.37))
+    (stroke (width 0) (type default))
+  )
+  (wire (pts (xy 300.99 54.61) (xy 303.53 54.61))
     (stroke (width 0) (type default))
   )
@@
         (path "/0ebd4cf3-0d07-4562-b8b5-7ef6838582db"
           (reference "#PWR038") (unit 1)
+        )
+      )
+    )
+  )
+  (symbol (lib_id "power:GND") (at 303.53 54.61 0) (unit 1)
+    (in_bom yes) (on_board yes) (dnp no) (fields_autoplaced)
+    (property "Reference" "#PWR039" (at 303.53 60.96 0)
+      (effects (font (size 1.27 1.27)) hide)
+    )
+    (property "Value" "GND" (at 303.53 59.69 0)
+      (effects (font (size 1.27 1.27)))
+    )
+    (property "Footprint" "" (at 303.53 54.61 0)
+      (effects (font (size 1.27 1.27)) hide)
+    )
+    (property "Datasheet" "" (at 303.53 54.61 0)
+      (effects (font (size 1.27 1.27)) hide)
+    )
+    (pin "1")
+    (instances
+      (project "C64-Pi1541"
+        (path "/0ebd4cf3-0d07-4562-b8b5-7ef6838582db"
+          (reference "#PWR039") (unit 1)
         )
       )
@@
         (path "/0ebd4cf3-0d07-4562-b8b5-7ef6838582db"
           (reference "JP2") (unit 1)
+        )
+      )
+    )
+  )
+  (symbol (lib_id "power:+5V") (at 314.96 36.83 0) (unit 1)
+    (in_bom yes) (on_board yes) (dnp no) (fields_autoplaced)
+    (property "Reference" "#PWR025" (at 314.96 40.64 0)
+      (effects (font (size 1.27 1.27)) hide)
+    )
+    (property "Value" "+5V" (at 314.96 33.02 0)
+      (effects (font (size 1.27 1.27)))
+    )
+    (property "Footprint" "" (at 314.96 36.83 0)
+      (effects (font (size 1.27 1.27)) hide)
+    )
+    (property "Datasheet" "" (at 314.96 36.83 0)
+      (effects (font (size 1.27 1.27)) hide)
+    )
+    (pin "1")
+    (instances
+      (project "C64-Pi1541"
+        (path "/0ebd4cf3-0d07-4562-b8b5-7ef6838582db"
+          (reference "#PWR025") (unit 1)
         )
       )
@@
         )
       )
+    )
+  )
+  (symbol (lib_id "Connector:USB_B_Micro") (at 303.53 44.45 0) (unit 1)
+    (in_bom yes) (on_board yes) (dnp no) (fields_autoplaced)
+    (property "Reference" "J5" (at 303.53 33.02 0)
+      (effects (font (size 1.27 1.27)))
+    )
+    (property "Value" "USB_B_Micro power" (at 303.53 35.56 0)
+      (effects (font (size 1.27 1.27)))
+    )
+    (property "Footprint" "Connector_USB:USB_Micro-B_Molex-105017-0001" (at 307.34 45.72 0)
+      (effects (font (size 1.27 1.27)) hide)
+    )
+    (property "Datasheet" "~" (at 307.34 45.72 0)
+      (effects (font (size 1.27 1.27)) hide)
+    )
+    (pin "1")
+    (pin "2")
+    (pin "3")
+    (pin "4")
+    (pin "5")
+    (pin "6")
+    (instances
+      (project "C64-Pi1541"
+        (path "/0ebd4cf3-0d07-4562-b8b5-7ef6838582db"
+          (reference "J5") (unit 1)
+        )
+      )

Commit message: C64-Cartridge : addition of EpyxFastload daughter board ; some silkscreen changes. C64-KungFuFlash, C64-Pi1541 : small updates before production. New C64-efuse board that fit inside the DIN plug.
Parts:
- U1: footprint Package_SO:SO-14_5.3x10.2mm_P1.27mm -> Package_DIP:DIP-14_W7.62mm
Connections:
- net CLK: now also U1.10; no longer U1.4
- net CLK_OUT: now also U1.11; no longer U1.3
- net DATA: now also U1.8; no longer U1.6
- net DATA_OUT: now also U1.9; no longer U1.5
- net GND: now also U1.1, U1.3, U1.5; no longer U1.11, U1.13, U1.9
- net SRQ: now also U1.12; no longer U1.2
- net SRQ_OUT: now also U1.13; no longer U1.1
Changed lines of the file:
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@@
     )
   )
-  (symbol (lib_id "74xx_IEEE:7406") (at 137.16 181.61 0) (unit 1)
+  (symbol (lib_id "74xx_IEEE:7406") (at 137.16 181.61 0) (unit 6)
     (in_bom yes) (on_board yes) (dnp no) (fields_autoplaced)
     (property "Reference" "U1" (at 147.32 178.4351 0)
@@
       (effects (font (size 1.27 1.27)))
     )
-    (property "Footprint" "Package_SO:SO-14_5.3x10.2mm_P1.27mm" (at 137.16 181.61 0)
+    (property "Footprint" "Package_DIP:DIP-14_W7.62mm" (at 137.16 181.61 0)
       (effects (font (size 1.27 1.27)) hide)
     )
@@
       (project "C64-Pi1541"
         (path "/0ebd4cf3-0d07-4562-b8b5-7ef6838582db"
-          (reference "U1") (unit 1)
+          (reference "U1") (unit 6)
         )
       )
@@
     )
   )
-  (symbol (lib_id "74xx_IEEE:7406") (at 137.16 151.13 0) (unit 2)
+  (symbol (lib_id "74xx_IEEE:7406") (at 137.16 151.13 0) (unit 5)
     (in_bom yes) (on_board yes) (dnp no) (fields_autoplaced)
     (property "Reference" "U1" (at 147.32 147.9551 0)
@@
       (effects (font (size 1.27 1.27)))
     )
-    (property "Footprint" "Package_SO:SO-14_5.3x10.2mm_P1.27mm" (at 137.16 151.13 0)
+    (property "Footprint" "Package_DIP:DIP-14_W7.62mm" (at 137.16 151.13 0)
       (effects (font (size 1.27 1.27)) hide)
     )
@@
       (project "C64-Pi1541"
         (path "/0ebd4cf3-0d07-4562-b8b5-7ef6838582db"
-          (reference "U1") (unit 2)
+          (reference "U1") (unit 5)
         )
       )
@@
     )
   )
-  (symbol (lib_id "power:PWR_FLAG") (at 50.8 92.71 90) (unit 1)
-    (in_bom yes) (on_board yes) (dnp no) (fields_autoplaced)
-    (property "Reference" "#FLG02" (at 48.895 92.71 0)
-      (effects (font (size 1.27 1.27)) hide)
-    )
-    (property "Value" "PWR_FLAG" (at 46.99 93.345 90)
-      (effects (font (size 1.27 1.27)) (justify left))
-    )
-    (property "Footprint" "" (at 50.8 92.71 0)
-      (effects (font (size 1.27 1.27)) hide)
-    )
-    (property "Datasheet" "~" (at 50.8 92.71 0)
-      (effects (font (size 1.27 1.27)) hide)
-    )
-    (pin "1")
-    (instances
-      (project "C64-Pi1541"
-        (path "/0ebd4cf3-0d07-4562-b8b5-7ef6838582db"
-          (reference "#FLG02") (unit 1)
-        )
-      )
-    )
-  )
   (symbol (lib_id "power:+3.3V") (at 198.12 143.51 0) (unit 1)
     (in_bom yes) (on_board yes) (dnp no) (fields_autoplaced)
@@
     )
   )
-  (symbol (lib_id "74xx_IEEE:7406") (at 77.47 181.61 0) (unit 6)
+  (symbol (lib_id "74xx_IEEE:7406") (at 77.47 181.61 0) (unit 1)
     (in_bom yes) (on_board yes) (dnp no) (fields_autoplaced)
     (property "Reference" "U1" (at 87.63 178.4351 0)
@@
       (effects (font (size 1.27 1.27)))
     )
-    (property "Footprint" "Package_SO:SO-14_5.3x10.2mm_P1.27mm" (at 77.47 181.61 0)
+    (property "Footprint" "Package_DIP:DIP-14_W7.62mm" (at 77.47 181.61 0)
       (effects (font (size 1.27 1.27)) hide)
     )
@@
       (project "C64-Pi1541"
         (path "/0ebd4cf3-0d07-4562-b8b5-7ef6838582db"
-          (reference "U1") (unit 6)
+          (reference "U1") (unit 1)
         )
       )
@@
     )
   )
-  (symbol (lib_id "74xx_IEEE:7406") (at 77.47 120.65 0) (unit 4)
+  (symbol (lib_id "74xx_IEEE:7406") (at 77.47 120.65 0) (unit 3)
     (in_bom yes) (on_board yes) (dnp no) (fields_autoplaced)
     (property "Reference" "U1" (at 87.63 117.4751 0)
@@
       (effects (font (size 1.27 1.27)))
     )
-    (property "Footprint" "Package_SO:SO-14_5.3x10.2mm_P1.27mm" (at 77.47 120.65 0)
+    (property "Footprint" "Package_DIP:DIP-14_W7.62mm" (at 77.47 120.65 0)
       (effects (font (size 1.27 1.27)) hide)
     )
@@
       (project "C64-Pi1541"
         (path "/0ebd4cf3-0d07-4562-b8b5-7ef6838582db"
-          (reference "U1") (unit 4)
+          (reference "U1") (unit 3)
         )
       )
@@
     )
   )
-  (symbol (lib_id "74xx_IEEE:7406") (at 137.16 120.65 0) (unit 3)
+  (symbol (lib_id "74xx_IEEE:7406") (at 137.16 120.65 0) (unit 4)
     (in_bom yes) (on_board yes) (dnp no) (fields_autoplaced)
     (property "Reference" "U1" (at 147.32 117.4751 0)
@@
       (effects (font (size 1.27 1.27)))
     )
-    (property "Footprint" "Package_SO:SO-14_5.3x10.2mm_P1.27mm" (at 137.16 120.65 0)
+    (property "Footprint" "Package_DIP:DIP-14_W7.62mm" (at 137.16 120.65 0)
       (effects (font (size 1.27 1.27)) hide)
     )
@@
       (project "C64-Pi1541"
         (path "/0ebd4cf3-0d07-4562-b8b5-7ef6838582db"
-          (reference "U1") (unit 3)
+          (reference "U1") (unit 4)
         )
       )
@@
     )
   )
-  (symbol (lib_id "power:PWR_FLAG") (at 55.88 26.67 90) (unit 1)
-    (in_bom yes) (on_board yes) (dnp no) (fields_autoplaced)
-    (property "Reference" "#FLG01" (at 53.975 26.67 0)
-      (effects (font (size 1.27 1.27)) hide)
-    )
-    (property "Value" "PWR_FLAG" (at 52.07 27.305 90)
-      (effects (font (size 1.27 1.27)) (justify left))
-    )
-    (property "Footprint" "" (at 55.88 26.67 0)
-      (effects (font (size 1.27 1.27)) hide)
-    )
-    (property "Datasheet" "~" (at 55.88 26.67 0)
-      (effects (font (size 1.27 1.27)) hide)
-    )
-    (pin "1")
-    (instances
-      (project "C64-Pi1541"
-        (path "/0ebd4cf3-0d07-4562-b8b5-7ef6838582db"
-          (reference "#FLG01") (unit 1)
-        )
-      )
-    )
-  )
   (symbol (lib_id "Mechanical:MountingHole") (at 19.05 146.05 0) (unit 1)
     (in_bom yes) (on_board yes) (dnp no) (fields_autoplaced)
@@
     )
   )
-  (symbol (lib_id "74xx_IEEE:7406") (at 77.47 151.13 0) (unit 5)
+  (symbol (lib_id "74xx_IEEE:7406") (at 77.47 151.13 0) (unit 2)
     (in_bom yes) (on_board yes) (dnp no) (fields_autoplaced)
     (property "Reference" "U1" (at 87.63 147.9551 0)
@@
       (effects (font (size 1.27 1.27)))
     )
-    (property "Footprint" "Package_SO:SO-14_5.3x10.2mm_P1.27mm" (at 77.47 151.13 0)
+    (property "Footprint" "Package_DIP:DIP-14_W7.62mm" (at 77.47 151.13 0)
       (effects (font (size 1.27 1.27)) hide)
     )
@@
       (project "C64-Pi1541"
         (path "/0ebd4cf3-0d07-4562-b8b5-7ef6838582db"
-          (reference "U1") (unit 5)
-        )
-      )
+          (reference "U1") (unit 2)
+        )
+      )
